File: hardware/Pico-Dev/picodev.brd (EAGLE design)
At the start: 63.5 x 63.5 mm, 5 parts

Commit message: Latest updates to match upstream firmware changes.
Parts:
- added PWR: (no value), pinhead:1X02
- renumbered JP1 to DEBUG
Connections:
- net A0: now also U$1.16; no longer U$1.15
- net A1: now also DEBUG.28, U$1.15
- net GND: now also PWR.1
- net VCC33: now also PWR.2; no longer DEBUG.28
Routing:
- net A1: track 0.00 -> 79.5 mm
- net VCC33: track 97.5 -> 88.8 mm
- net A0: track 72.1 -> 75.7 mm
- net D4: track 59.4 -> 61.5 mm
- net D5: track 58.2 -> 60.3 mm
- net D6: track 51.5 -> 53.6 mm
- net D7: track 50.7 -> 52.8 mm
- net D3: track 70.9 -> 72.0 mm
Other:
- board text added: "A1"
- board text removed: "3v3"
