File: hardware/Pico-Dev/picodev.sch (EAGLE design)
At the start: 5 parts

Commit message: Latest updates to match upstream firmware changes.
Parts:
- added PWR: (no value), pinhead:PINHD-1X2
- renumbered JP1 to DEBUG
Connections:
- net A0: now also U$1.GP15; no longer U$1.GP14
- net A1: now also DEBUG.28, U$1.GP14
- net GND: now also PWR.1
- net VCC33: now also PWR.2; no longer DEBUG.28
